File: PCB/CybdoClock.kicad_sch (KiCad schematic)
At the start: 237 parts, among them Q1 CJL2301, Q10 HSW6822, Q11 HSW6822, Q12 HSW6822, Q13 HSW6822, Q14 HSW6822, Q2 CJL2301, Q3 CJL2301, Q4 CJL2301, Q5 CJL2301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

Commit message: use built in serial pins, start on firmware using circuitpython
Connections:
- net CLOCK: now also U1.9 (GPIO19_D8_SCK); no longer U1.5 (GPIO22_D4_SDA)
- net DATA: now also U1.11 (GPIO18_D10_MOSI); no longer U1.3 (GPIO2_A2_D2)
Changed lines of the file:
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@@
 	)
 	(no_connect
-		(at 389.89 60.96)
+		(at 293.37 222.25)
 	)
 	(no_connect
-		(at 293.37 222.25)
+		(at 351.79 57.15)
 	)
 	(no_connect
@@
 	)
 	(no_connect
+		(at 351.79 49.53)
+	)
+	(no_connect
 		(at 351.79 45.72)
 	)
@@
 	)
 	(no_connect
-		(at 389.89 53.34)
-	)
-	(no_connect
 		(at 293.37 227.33)
 	)
@@
 	(wire
 		(pts
+			(xy 389.89 60.96) (xy 400.05 60.96)
+		)
+		(stroke
+			(width 0)
+			(type default)
+		)
+	)
+	(wire
+		(pts
 			(xy 196.85 97.79) (xy 196.85 130.81)
 		)
@@
 	(wire
 		(pts
-			(xy 339.09 57.15) (xy 351.79 57.15)
-		)
-		(stroke
-			(width 0)
-			(type default)
-		)
-	)
-	(wire
-		(pts
 			(xy 88.9 259.08) (xy 111.76 259.08)
 		)
@@
 	(wire
 		(pts
+			(xy 389.89 53.34) (xy 400.05 53.34)
+		)
+		(stroke
+			(width 0)
+			(type default)
+		)
+	)
+	(wire
+		(pts
 			(xy 138.43 196.85) (xy 139.7 196.85)
 		)
@@
 	(wire
 		(pts
-			(xy 389.89 45.72) (xy 394.97 45.72)
+			(xy 389.89 45.72) (xy 419.1 45.72)
 		)
 		(stroke
@@
 	(wire
 		(pts
-			(xy 339.09 49.53) (xy 351.79 49.53)
-		)
-		(stroke
-			(width 0)
-			(type default)
-		)
-	)
-	(wire
-		(pts
 			(xy 167.64 58.42) (xy 179.07 58.42)
 		)
@@
 	(wire
 		(pts
-			(xy 394.97 45.72) (xy 394.97 71.12)
+			(xy 419.1 45.72) (xy 419.1 68.58)
 		)
 		(stroke
@@
 		)
 	)
-	(label "DATA"
-		(at 339.09 49.53 0)
-		(effects
-			(font
-				(size 1.27 1.27)
-			)
-			(justify left bottom)
-		)
-	)
 	(label "CLOCK"
 		(at 262.89 25.4 270)
@@
 		)
 	)
+	(label "CLOCK"
+		(at 400.05 60.96 180)
+		(effects
+			(font
+				(size 1.27 1.27)
+			)
+			(justify right bottom)
+		)
+	)
 	(label "COL5"
 		(at 304.8 209.55 180)
@@
 		)
 	)
-	(label "CLOCK"
-		(at 339.09 57.15 0)
-		(effects
-			(font
-				(size 1.27 1.27)
-			)
-			(justify left bottom)
-		)
-	)
 	(label "COL11"
 		(at 200.66 292.1 90)
@@
 		)
 	)
+	(label "DATA"
+		(at 400.05 53.34 180)
+		(effects
+			(font
+				(size 1.27 1.27)
+			)
+			(justify right bottom)
+		)
+	)
 	(label "ROW6"
 		(at 25.4 102.87 0)
@@
 	(symbol
 		(lib_id "power:GND")
-		(at 394.97 71.12 0)
+		(at 419.1 68.58 0)
 		(unit 1)
 		(body_style 1)
@@
 		(fields_autoplaced yes)
 		(property "Reference" "#PWR02"
-			(at 394.97 77.47 0)
+			(at 419.1 74.93 0)
 			(hide yes)
 			(show_name no)
@@
 		)
 		(property "Value" "GND"
-			(at 394.97 76.2 0)
+			(at 419.1 73.66 0)
 			(show_name no)
 			(do_not_autoplace no)
@@
 		)
 		(property "Footprint" ""
-			(at 394.97 71.12 0)
+			(at 419.1 68.58 0)
 			(hide yes)
 			(show_name no)
@@
 		)
 		(property "Datasheet" ""
-			(at 394.97 71.12 0)
+			(at 419.1 68.58 0)
 			(hide yes)
 			(show_name no)
@@
 		)
 		(property "Description" "Power symbol creates a global label with name \"GND\" , ground"
-			(at 394.97 71.12 0)
+			(at 419.1 68.58 0)
 			(hide yes)
 			(show_name no)
